File: TrActor-Board.kicad_sch (KiCad schematic)
At the start: 24 parts, among them J3 GCT4720, J4 Batt, J5 NTC, SW1 Power, SW2 Reset, U3 LSM6DSO32, U6 USBLC6-2P6

Commit message: routing hell
Parts:
- removed JP1: Reset, Connector_PinHeader_2.54mm:PinHeader_1x02_P2.54mm_Vertical_SMD_Pin1Left, symbol Jumper:Jumper_2_Open
- removed SW2: Reset, Button_Switch_SMD:SW_SPST_EVQP7A, symbol Switch:SW_Push
- removed TP11: BTN_RESET, TestPoint:TestPoint_Pad_D1.5mm, symbol Connector:TestPoint
- removed U3: LSM6DSO32, Package_LGA:LGA-14_3x2.5mm_P0.5mm_LayoutBorder3x4y, symbol Sensor_Motion:LSM6DS3
- added H1, H2, H3: M2, MountingHole:MountingHole_2.2mm_M2_DIN965_Pad_TopBottom, symbol Mechanical:MountingHole_Pad
- added U3: ICM-40609, Sensor_Motion:InvenSense_QFN-24_3x3mm_P0.4mm, symbol TrActor:ICM-40609
- TP10, TP13, TP14, TP22, TP23: footprint TestPoint:TestPoint_Pad_D1.5mm -> TestPoint:TestPoint_Pad_D1.0mm
- TP12, TP5, TP9: footprint TestPoint:TestPoint_Pad_1.5x1.5mm -> TestPoint:TestPoint_Pad_1.0x1.0mm
Connections:
- net +1V8: now also U3.13 (VDD), U3.8 (VDDIO)
- net BTN_POWER: now also SW1.1; no longer SW1.2
- net CS_IMU: now also U3.22 (~{CS})
- net GND: now also SW1.2, U3.11 (RESV), U3.18 (GND), U3.20 (RESV); no longer SW1.1
- net IMU_INT1: now also U3.12 (INT1)
- net IMU_INT2: now also U3.19 (INT2)
- net MISO: now also U3.9 (SDO)
- net MOSI: now also U3.24 (SDI)
- net SCK: now also U3.23 (SCLK)
- new net: U3.1 (NC), U3.10 (NC), U3.14 (NC), U3.15 (NC), U3.16 (NC), U3.17 (NC), U3.2 (NC), U3.21 (NC), U3.3 (NC), U3.4 (NC), U3.5 (NC), U3.6 (NC), U3.7 (NC)
- no-connect marks 4 -> 7
Other:
- note added: "TO:DO:"
- note removed: "TO:DO: - NTC connector footprint selection"
- moved on the sheet: C19, TP22, TP23

Commit message: ready for DR
Parts:
- removed TP13: D-, TestPoint:TestPoint_Pad_D1.0mm, symbol Connector:TestPoint
- removed TP14: D+, TestPoint:TestPoint_Pad_D1.0mm, symbol Connector:TestPoint
- added SW2: Reset, Button_Switch_SMD:SW_SPST_EVQP7A, symbol Switch:SW_Push
- added TP11: BTN_RESET, TestPoint:TestPoint_Pad_D1.0mm, symbol Connector:TestPoint
Connections:
- net GND: now also SW2.2
- net BATT_RAW: now reaches F2.1, J4.1 (Pin_1), TP9.1
- net USB_D+: now reaches J3.A6 (D+), J3.B6 (D+), U6.3 (I/O2)
- net USB_D-: now reaches J3.A7 (D-), J3.B7 (D-), U6.1 (I/O1)
- net D+: now reaches R11.2, U6.4 (I/O2)
- net D-: now reaches R12.1, U6.6 (I/O1)
- new net BTN_RESET: SW2.1, TP11.1
