File: TrActor-Board.kicad_pcb (KiCad board)
At the start: 4 copper layers, 0 parts

Commit message: schematic & bom done except for UWB RF
Parts:
- added C1: 0.1u, Capacitor_SMD:C_0402_1005Metric, F.Cu at (131.4, 69.8)
- added C10: 1u, Capacitor_SMD:C_0402_1005Metric, F.Cu at (134.3, 73.8)
- added C11: 0.1u, Capacitor_SMD:C_0402_1005Metric, F.Cu at (134.3, 75.7)
- added C12: 0.1u, Capacitor_SMD:C_0402_1005Metric, F.Cu at (134.3, 77.7)
- added C13: 0.1u, Capacitor_SMD:C_0402_1005Metric, F.Cu at (134.3, 79.7)
- added C14: 4.7n, Capacitor_SMD:C_0402_1005Metric, F.Cu at (158.0, 103.0)
- added C15: 12p, Capacitor_SMD:C_0402_1005Metric, F.Cu at (134.3, 81.7)
- added C16: 12p, Capacitor_SMD:C_0402_1005Metric, F.Cu at (137.2, 69.8)
- added C17: 1.0p, Capacitor_SMD:C_0402_1005Metric, F.Cu at (137.2, 71.8)
- added C18: 1.2p, Capacitor_SMD:C_0402_1005Metric, F.Cu at (137.2, 73.8)
- added C19: 0.1u, Capacitor_SMD:C_0402_1005Metric, F.Cu at (158.0, 105.0)
- added C2: 100p, Capacitor_SMD:C_0402_1005Metric, F.Cu at (131.4, 71.8)
- added C20: 0.1u, Capacitor_SMD:C_0402_1005Metric, F.Cu at (135.4, 92.9)
- added C21: 0.1u, Capacitor_SMD:C_0402_1005Metric, F.Cu at (135.4, 94.8)
- added C22: 4.7n, Capacitor_SMD:C_0402_1005Metric, F.Cu at (135.4, 96.8)
- added C23: 10u, Capacitor_SMD:C_0603_1608Metric, F.Cu at (132.0, 93.1)
- added C24: 4.7n, Capacitor_SMD:C_0402_1005Metric, F.Cu at (138.3, 92.9)
- added C25: 0.1u, Capacitor_SMD:C_0402_1005Metric, F.Cu at (138.3, 94.8)
- added C26: 10u, Capacitor_SMD:C_0603_1608Metric, F.Cu at (132.0, 95.7)
- added C27: 4.7n, Capacitor_SMD:C_0402_1005Metric, F.Cu at (138.3, 96.8)
- added C28: 0.1u, Capacitor_SMD:C_0402_1005Metric, F.Cu at (141.2, 92.9)
- added C29: 0.1u, Capacitor_SMD:C_0402_1005Metric, F.Cu at (141.2, 94.8)
- added C3: 4.7u, Capacitor_SMD:C_0402_1005Metric, F.Cu at (131.4, 73.8)
- added C30: 2200p, Capacitor_SMD:C_0402_1005Metric, F.Cu at (141.2, 96.8)
- added C31: 1u, Capacitor_SMD:C_0402_1005Metric, F.Cu at (166.7, 69.8)
- added C32: 1u, Capacitor_SMD:C_0402_1005Metric, F.Cu at (166.7, 71.8)
- added C33: 10u, Capacitor_SMD:C_0603_1608Metric, F.Cu at (155.2, 70.1)
- added C34: 10u, Capacitor_SMD:C_0603_1608Metric, F.Cu at (155.2, 72.6)
- added C35: 10u, Capacitor_SMD:C_0603_1608Metric, F.Cu at (155.2, 75.1)
- added C36: 10u, Capacitor_SMD:C_0603_1608Metric, F.Cu at (155.2, 77.6)
- added C37: 10u, Capacitor_SMD:C_0603_1608Metric, F.Cu at (155.2, 80.1)
- added C38: 0.1u, Capacitor_SMD:C_0402_1005Metric, F.Cu at (166.7, 73.8)
- added C39: 2.2u, Capacitor_SMD:C_0603_1608Metric, F.Cu at (159.2, 70.1)
- added C4: 4.7u, Capacitor_SMD:C_0402_1005Metric, F.Cu at (131.4, 75.7)
- added C41: TBD, Capacitor_SMD:C_0402_1005Metric, F.Cu at (137.2, 75.7)
- added C42: TBD, Capacitor_SMD:C_0402_1005Metric, F.Cu at (137.2, 77.7)
- added C5: 4.7u, Capacitor_SMD:C_0402_1005Metric, F.Cu at (131.4, 77.7)
- added C6: 820p, Capacitor_SMD:C_0402_1005Metric, F.Cu at (131.4, 79.7)
- added C7: 1u, Capacitor_SMD:C_0402_1005Metric, F.Cu at (131.4, 81.7)
- added C8: 47n, Capacitor_SMD:C_0402_1005Metric, F.Cu at (134.3, 69.8)
- added C9: TBD, Capacitor_SMD:C_0402_1005Metric, F.Cu at (134.3, 71.8)
- added D1: RX,Orange, LED_SMD:LED_0603_1608Metric, F.Cu at (143.7, 99.1)
- added D2: TX,White, LED_SMD:LED_0603_1608Metric, F.Cu at (143.7, 101.7)
- added D3: BLUE, LED_SMD:LED_0603_1608Metric, F.Cu at (148.5, 85.1)
- added D4: Green, LED_SMD:LED_0603_1608Metric, F.Cu at (163.2, 70.1)
- added D5: Yellow, LED_SMD:LED_0603_1608Metric, F.Cu at (163.2, 72.7)
- added D6: Red, LED_SMD:LED_0603_1608Metric, F.Cu at (163.2, 75.3)
- added F1: 500mA 6V, Fuse:Fuse_0603_1608Metric, F.Cu at (149.7, 103.3)
- added F2: 500mA 6V, Fuse:Fuse_0603_1608Metric, F.Cu at (149.7, 105.8)
- added FB1: BLM15PX330SZ1D, Inductor_SMD:L_0603_1608Metric, F.Cu at (132.0, 98.2)
- added J1: TagConnect, Connector:Tag-Connect_TC2030-IDC-NL_2x03_P1.27mm_Vertical, F.Cu at (142.6, 81.3)
- added J2: Conn_ARM_JTAG_SWD_10, Connector_PinHeader_1.27mm:PinHeader_2x05_P1.27mm_Vertical_SMD, F.Cu at (146.3, 73.1)
- added J3: GCT4720, TrActor:GCT_USB4720-03-A_REVA, F.Cu at (187.8, 124.5)
- added L1: 10u, Inductor_SMD:L_0603_1608Metric, F.Cu at (140.6, 85.1)
- added L2: 15n, Inductor_SMD:L_0402_1005Metric, F.Cu at (140.1, 69.8)
- added L3: 4.7n, Inductor_SMD:L_0402_1005Metric, F.Cu at (140.1, 71.8)
- added L4: 2.2n, Inductor_SMD:L_0402_1005Metric, F.Cu at (140.1, 73.8)
- added L5: 2.2u, Inductor_SMD:L_0805_2012Metric, F.Cu at (155.4, 82.8)
- added L6: 2.2u, Inductor_SMD:L_0805_2012Metric, F.Cu at (155.4, 85.5)
- added Q1: NMOS, Package_TO_SOT_SMD:SOT-363_SC-70-6, F.Cu at (140.0, 106.9)
- added R1: 50R0, Resistor_SMD:R_0402_1005Metric, F.Cu at (143.5, 106.0)
- added R10: 68k, Resistor_SMD:R_0603_1608Metric, F.Cu at (159.2, 80.1)
- added R11: 0R, Resistor_SMD:R_0402_1005Metric, F.Cu at (163.0, 92.9)
- added R12: 0R, Resistor_SMD:R_0402_1005Metric, F.Cu at (163.0, 94.9)
- added R13: 1M, Resistor_SMD:R_0402_1005Metric, F.Cu at (163.0, 96.9)
- added R14: 0R, Resistor_SMD:R_0402_1005Metric, F.Cu at (140.1, 75.8)
- added R15: 0R, Resistor_SMD:R_0402_1005Metric, F.Cu at (140.1, 77.8)
- added R2: 1k, Resistor_SMD:R_0603_1608Metric, F.Cu at (132.0, 100.7)
- added R3: 1k, Resistor_SMD:R_0603_1608Metric, F.Cu at (132.0, 103.2)
- added R4: 330, Resistor_SMD:R_0603_1608Metric, F.Cu at (132.0, 105.7)
- added R5: 330, Resistor_SMD:R_0603_1608Metric, F.Cu at (132.0, 108.2)
- added R6: 330, Resistor_SMD:R_0603_1608Metric, F.Cu at (140.6, 87.6)
- added R7: 10k, Resistor_SMD:R_0603_1608Metric, F.Cu at (159.2, 72.6)
- added R8: 10k, Resistor_SMD:R_0603_1608Metric, F.Cu at (159.2, 75.1)
- added R9: 47k, Resistor_SMD:R_0603_1608Metric, F.Cu at (159.2, 77.6)
- added U1: nRF52833_QDxx, Package_DFN_QFN:QFN-40-1EP_5x5mm_P0.4mm_EP3.6x3.6mm, F.Cu at (134.0, 86.3)
- added U2: DW3210, TrActor:QFN-40-1EP_5x5mm_P0.4mm, F.Cu at (138.0, 101.4)
- added U3: LSM6DSO32, Package_LGA:LGA-14_3x2.5mm_P0.5mm_LayoutBorder3x4y, F.Cu at (154.3, 104.1)
- added U4: ATX-13, Crystal:Crystal_SMD_2016-4Pin_2.0x1.6mm, F.Cu at (136.0, 106.9)
- added U5: nPM1300, Package_DFN_QFN:QFN-40-1EP_5x5mm_P0.4mm_EP3.6x3.6mm_ThermalVias, F.Cu at (171.6, 82.7)
- added U6: USBLC6-2P6, Package_TO_SOT_SMD:SOT-666, F.Cu at (161.5, 103.9)
- added Y1: 32MHz, Oscillator:Oscillator_SMD_ECS_2520MV-xxx-xx-4Pin_2.5x2.0mm, F.Cu at (144.5, 86.0)
- added Y2: 32.768k, Crystal:Crystal_SMD_2012-2Pin_2.0x1.2mm, F.Cu at (148.5, 88.1)
Other:
- board outline added: 31.8 x 44.4 mm

Commit message: routing started
Parts:
- removed L4: 2.2n, Inductor_SMD:L_0402_1005Metric
- added AE1: NFC, TrActor:NFC-Coil, F.Cu at (125.4, 196.8)
- added AE2: SR4W035, TrActor:SR4W035_4X6_ANT, F.Cu at (261.8, 37.9)
- added C40: 2.0p, Capacitor_SMD:C_0402_1005Metric, F.Cu at (36.3, 103.2)
- added C43: 0.22u, Capacitor_SMD:C_0402_1005Metric, F.Cu at (35.7, 108.8)
- added C44: 47u, Capacitor_SMD:CP_Elec_5x5.8, F.Cu at (23.6, 99.2)
- added C45: 47u, Capacitor_SMD:CP_Elec_5x5.8, F.Cu at (25.3, 107.9)
- added FB2: TBD, Inductor_SMD:L_0603_1608Metric, F.Cu at (31.8, 106.4)
- added J4: Batt, Connector_JST:JST_PH_S2B-PH-SM4-TB_1x02-1MP_P2.00mm_Horizontal, F.Cu at (34.0, 182.8)
- added J5: NTC, Connector_JST:JST_SH_SM02B-SRSS-TB_1x02-1MP_P1.00mm_Horizontal, F.Cu at (43.7, 184.7)
- added JP1: Reset, Connector_PinHeader_2.54mm:PinHeader_1x02_P2.54mm_Vertical_SMD_Pin1Left, F.Cu at (36.5, 41.7)
- added JP2: RF_GND_BRIDGE, Jumper:SolderJumper-2_P1.3mm_Bridged2Bar_RoundedPad1.0x1.5mm, F.Cu at (30.6, 119.0)
- added R16: 10k, Resistor_SMD:R_0402_1005Metric, F.Cu at (55.2, 112.0)
- added R17: 10k, Resistor_SMD:R_0402_1005Metric, F.Cu at (55.2, 114.5)
- added SW1: Power, Button_Switch_SMD:SW_SPST_EVQP7A, F.Cu at (36.1, 29.6)
- added SW2: Reset, Button_Switch_SMD:SW_SPST_EVQP7A, F.Cu at (36.1, 34.7)
- added U7: USBLC6-2P6, Package_TO_SOT_SMD:SOT-666, F.Cu at (228.4, 29.7)
- C17: value 1.0p -> 1.5p
- C41, C42: value TBD -> 120pF,TBD
- J2: value Conn_ARM_JTAG_SWD_10 -> Debug
- L3: value 4.7n -> 4.2n
- R10, R2, R3, R4, R5, R6, R7, R8, R9: footprint Resistor_SMD:R_0603_1608Metric -> Resistor_SMD:R_0402_1005Metric
- U5: footprint Package_DFN_QFN:QFN-40-1EP_5x5mm_P0.4mm_EP3.6x3.6mm_ThermalVias -> Package_DFN_QFN:QFN-32-1EP_5x5mm_P0.5mm_EP3.45x3.45mm_ThermalVias
- moved F2 142.9 mm to (35.2, 191.4)
- moved C13 133.7 mm to (259.4, 32.6), turned to 90 degrees
- moved C2 131.3 mm to (257.3, 34.6)
- moved C7 129.8 mm to (250.8, 30.7)
- moved C6 129.5 mm to (254.7, 40.0), turned to -90 degrees
- moved C9 128.2 mm to (257.3, 35.5)
- moved C12 128.0 mm to (254.4, 33.5), turned to 90 degrees
- moved C18 127.1 mm to (258.9, 37.0), turned to 90 degrees
- moved U1 127.0 mm to (251.0, 36.9)
- moved D4 125.2 mm to (43.3, 34.0)
- moved D5 125.2 mm to (43.3, 36.6)
- moved D6 125.2 mm to (43.3, 39.2)
- moved R1 124.8 mm to (19.2, 118.0)
- moved Y1 124.8 mm to (257.3, 32.6), turned to -90 degrees
- moved C41 124.5 mm to (133.5, 200.2)
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Connections:
- net Net-(D4-K) renamed /Power Management/GREEN
- net Net-(D5-K) renamed /Power Management/YELLOW
- net Net-(D6-K) renamed /Power Management/RED
- net Net-(U6-VBUS) renamed V_PRE
- C17 pad 1: Net-(U1-ANT) -> /MCU/ANT_BLE
- C41 pad 1: /MCU/NFC2 -> Net-(AE1-Pad2)
- C42 pad 2: /MCU/NFC1 -> Net-(AE1-Pad1)
- L1 pad 1: Net-(U1-DEC4) -> Net-(U1-DCC)
- L2 pad 2: Net-(U1-DCC) -> Net-(U1-DEC4)
- L3 pad 2: Net-(U1-ANT) -> /MCU/ANT_BLE
- R14 pad 1: /MCU/NFC1 -> /MCU/NFC+
- R15 pad 1: /MCU/NFC2 -> /MCU/NFC-
- U1 pad 22: /MCU/NFC1 -> /MCU/NFC+
- U1 pad 23: /MCU/NFC2 -> /MCU/NFC-
- U1 pad 24: Net-(U1-ANT) -> /MCU/ANT_BLE
- U2 pad 27: (no net) -> Net-(U2-VTX_D)
- U5 pad 23: USB_CC1 -> Net-(U5-CC1)
- U5 pad 24: USB_CC2 -> Net-(U5-CC2)
- U5 pad 6: (no net) -> GND
Routing:
- net GND: track 0.00 -> 58.1 mm, vias 0 -> 9
- net +1V8: track 0.00 -> 31.8 mm, vias 0 -> 6
- net Net-(J3-SHIELD): track 0.00 -> 27.9 mm
- net V_PRE: track 0.00 -> 12.3 mm
- net VSYS: track 0.00 -> 9.68 mm
- net Net-(U1-DEC4): track 0.00 -> 8.95 mm, vias 0 -> 1
- net NTC: track 0.00 -> 6.81 mm
- net MOSI: track 0.00 -> 6.36 mm
- net MISO: track 0.00 -> 6.12 mm
- net Net-(U1-XL2/P0.01): track 0.00 -> 6.11 mm
- net +BATT: track 0.00 -> 6.09 mm
- net VBUS: track 0.00 -> 6.08 mm
- net SCK: track 0.00 -> 5.99 mm
- net CS_DW: track 0.00 -> 5.80 mm
- net DW_WAKEUP: track 0.00 -> 5.33 mm
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Other:
- board size 31.8 x 44.4 mm -> 10.6 x 5 mm
- board text added: "TO:DO: - Route DW3000 area - Figure out actually good NFC antenna - Figure out UWB antenna - increase power trace widths - actual RF trace width calcs - physical layout (buttons, LEDs, etc)"

Commit message: routing hell
Parts:
- removed FB2: TBD, Inductor_SMD:L_0603_1608Metric
- removed JP1: Reset, Connector_PinHeader_2.54mm:PinHeader_1x02_P2.54mm_Vertical_SMD_Pin1Left
- removed JP2: RF_GND_BRIDGE, Jumper:SolderJumper-2_P1.3mm_Bridged2Bar_RoundedPad1.0x1.5mm
- removed SW2: Reset, Button_Switch_SMD:SW_SPST_EVQP7A
- added AE3: ACR0301U, Inductor_SMD:L_1206_3216Metric, F.Cu at (139.5, 73.7)
- added H1: M2, MountingHole:MountingHole_2.2mm_M2_DIN965_Pad_TopBottom, F.Cu at (139.5, 127.5)
- added H2: M2, MountingHole:MountingHole_2.2mm_M2_DIN965_Pad_TopBottom, F.Cu at (160.5, 72.5)
- added H3: M2, MountingHole:MountingHole_2.2mm_M2_DIN965_Pad_TopBottom, F.Cu at (160.5, 127.5)
- added TP1: VBUS, TestPoint:TestPoint_Pad_1.0x1.0mm, F.Cu at (-17.3, 91.1)
- added TP10: BTN_POWER, TestPoint:TestPoint_Pad_D1.0mm, F.Cu at (-28.4, 97.2)
- added TP12: GND, TestPoint:TestPoint_Pad_1.0x1.0mm, F.Cu at (-25.4, 94.2)
- added TP13: D-, TestPoint:TestPoint_Pad_D1.0mm, F.Cu at (-25.4, 97.2)
- added TP14: D+, TestPoint:TestPoint_Pad_D1.0mm, F.Cu at (-22.3, 91.1)
- added TP15: MOSI, TestPoint:TestPoint_Pad_D1.0mm, F.Cu at (-11.4, 75.4)
- added TP16: MISO, TestPoint:TestPoint_Pad_D1.0mm, F.Cu at (-11.4, 78.5)
- added TP17: SCK, TestPoint:TestPoint_Pad_D1.0mm, F.Cu at (-11.4, 81.5)
- added TP18: SDA, TestPoint:TestPoint_Pad_D1.0mm, F.Cu at (-11.4, 84.6)
- added TP19: SCL, TestPoint:TestPoint_Pad_D1.0mm, F.Cu at (-8.32, 75.4)
- added TP2: VSYS, TestPoint:TestPoint_Pad_1.0x1.0mm, F.Cu at (-17.3, 94.2)
- added TP20: CS_IMU, TestPoint:TestPoint_Pad_D1.0mm, F.Cu at (-8.32, 78.5)
- added TP21: CS_DW, TestPoint:TestPoint_Pad_D1.0mm, F.Cu at (-8.32, 81.5)
- added TP22: IMU_INT1, TestPoint:TestPoint_Pad_D1.0mm, F.Cu at (-22.3, 94.2)
- added TP23: IMU_INT2, TestPoint:TestPoint_Pad_D1.0mm, F.Cu at (-22.3, 97.2)
- added TP24: DW_WAKEUP, TestPoint:TestPoint_Pad_D1.0mm, F.Cu at (-19.5, 78.5)
- added TP25: DW_RST, TestPoint:TestPoint_Pad_D1.0mm, F.Cu at (-19.5, 81.5)
- added TP26: DW_IRQ, TestPoint:TestPoint_Pad_D1.0mm, F.Cu at (-19.5, 84.6)
- added TP27: RX, TestPoint:TestPoint_Pad_D1.0mm, F.Cu at (-16.4, 75.4)
- added TP28: TX, TestPoint:TestPoint_Pad_D1.0mm, F.Cu at (-16.4, 78.5)
- added TP29: SYNC, TestPoint:TestPoint_Pad_D1.0mm, F.Cu at (-16.4, 81.5)
- added TP3: +1.8V, TestPoint:TestPoint_Pad_1.0x1.0mm, F.Cu at (-14.2, 91.1)
- added TP4: +2.5V, TestPoint:TestPoint_Pad_1.0x1.0mm, F.Cu at (-14.2, 94.2)
- added TP5: VUSB, TestPoint:TestPoint_Pad_1.0x1.0mm, F.Cu at (-28.4, 91.1)
- added TP6: CC1, TestPoint:TestPoint_Pad_D1.0mm, F.Cu at (-11.2, 91.1)
- added TP7: CC2, TestPoint:TestPoint_Pad_D1.0mm, F.Cu at (-11.2, 94.2)
- added TP8: DW_EXTON, TestPoint:TestPoint_Pad_D1.0mm, F.Cu at (-19.5, 75.4)
- added TP9: BATT, TestPoint:TestPoint_Pad_1.0x1.0mm, F.Cu at (-28.4, 94.2)
- added Z1: OC, Inductor_SMD:L_0402_1005Metric, F.Cu at (141.1, 58.7)
- added Z2: 0R, Inductor_SMD:L_0402_1005Metric, F.Cu at (141.1, 60.7)
- added Z3: OC, Inductor_SMD:L_0402_1005Metric, F.Cu at (141.1, 62.7)
- U3: value LSM6DSO32 -> ICM-40609; footprint Package_LGA:LGA-14_3x2.5mm_P0.5mm_LayoutBorder3x4y -> Sensor_Motion:InvenSense_QFN-24_3x3mm_P0.4mm
- moved C44 223.2 mm to (241.1, 149.5)
- moved C45 221.1 mm to (241.1, 156.3)
- moved SW1 151.7 mm to (161.5, 115.0), turned to 90 degrees
- moved C39 147.5 mm to (149.8, 117.2), turned to -90 degrees
- moved C33 147.3 mm to (151.6, 117.2), turned to -90 degrees
- moved C31 146.5 mm to (152.8, 116.7), turned to -90 degrees
- moved C32 146.4 mm to (153.8, 116.7), turned to -90 degrees
- moved R9 144.9 mm to (147.9, 114.8), turned to 180 degrees
- moved R10 143.4 mm to (147.9, 113.8), turned to 180 degrees
- moved R8 141.6 mm to (147.9, 112.8), turned to 180 degrees
- moved R7 140.2 mm to (147.9, 111.8), turned to 180 degrees
- moved D4 139.8 mm to (162.0, 108.0), turned to 90 degrees
- moved U5 139.7 mm to (152.4, 111.9), turned to -90 degrees
- moved C38 138.6 mm to (147.9, 110.7), turned to 180 degrees
- moved D2 138.2 mm to (175.7, 52.8)
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Connections:
- C40 pad 2: unconnected-(C40-Pad2) -> Net-(C40-Pad2)
- R1 pad 1: /UWB/RF_UWB_GND -> GND
- SW1 pad 1: GND -> BTN_POWER
- SW1 pad 2: BTN_POWER -> GND
- U2 pad 10: /UWB/RF_UWB_GND -> GND
- U2 pad 11: /UWB/RF_UWB_GND -> GND
- U2 pad 12: /UWB/RF_UWB_GND -> GND
- U2 pad 14: /UWB/RF_UWB_GND -> GND
- U2 pad 15: /UWB/RF_UWB_GND -> GND
- U2 pad 16: /UWB/RF_UWB_GND -> GND
- U2 pad 17: /UWB/RF_UWB_GND -> GND
- U2 pad 19: /UWB/RF_UWB_GND -> GND
- U2 pad 20: /UWB/RF_UWB_GND -> GND
- U3 pad 1: MISO -> unconnected-(U3-NC-Pad1)
- U3 pad 11: unconnected-(U3-NC-Pad11) -> GND
- U3 pad 12: CS_IMU -> IMU_INT1
- U3 pad 13: SCK -> +1V8
- U3 pad 14: MOSI -> unconnected-(U3-NC-Pad14)
- U3 pad 2: GND -> unconnected-(U3-NC-Pad2)
- U3 pad 3: GND -> unconnected-(U3-NC-Pad3)
- U3 pad 4: IMU_INT1 -> unconnected-(U3-NC-Pad4)
- U3 pad 5: +1V8 -> unconnected-(U3-NC-Pad5)
- U3 pad 6: GND -> unconnected-(U3-NC-Pad6)
- U3 pad 7: GND -> unconnected-(U3-NC-Pad7)
- U3 pad 9: IMU_INT2 -> MISO
Routing:
- net GND: track 58.1 -> 128.4 mm, vias 9 -> 34
- net Net-(U5-CC1): track 2.37 -> 11.9 mm
- net Net-(U5-CC2): track 2.14 -> 10.7 mm
- net +2V5: track 3.48 -> 11.3 mm, vias 2 -> 3
- net /UWB/TXLED: track 0.00 -> 6.23 mm
- net /UWB/RXLED: track 0.00 -> 5.91 mm
- net Net-(U4-OUT): track 0.00 -> 5.01 mm
- net NTC: track 6.81 -> 1.90 mm, vias 0 -> 1
- net +1V8: track 31.8 -> 35.9 mm, vias 6 -> 9
- net Net-(U2-VDD2a): track 0.00 -> 4.04 mm
- net Net-(J4-Pin_1): track 0.00 -> 3.66 mm
- net VSYS: track 9.68 -> 6.09 mm, vias 0 -> 1
- net /UWB/RF_UWB: track 0.00 -> 3.23 mm
- net BTN_RESET: track 3.84 -> 1.64 mm, vias 0 -> 1
- net SCL: track 5.01 -> 2.85 mm
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- added copper zone on In1.Cu, net GND
Other:
- board size 10.6 x 5 mm -> 26 x 60 mm
- board text added: "TO:DO: - Figure out actually good NFC antenna - increase power trace widths - actual RF trace width calcs - physical layout (buttons, LEDs, etc)"
- board text removed: "TO:DO: - Route DW3000 area - Figure out actually good NFC antenna - Figure out UWB antenna - increase power trace widths - actual RF trace width calcs - physical layout (buttons, LEDs, etc)"

Commit message: ready for DR
Parts:
- removed R14, R15: 0R, Resistor_SMD:R_0402_1005Metric
- removed TP13: D-, TestPoint:TestPoint_Pad_D1.0mm
- removed TP14: D+, TestPoint:TestPoint_Pad_D1.0mm
- removed TP6: CC1, TestPoint:TestPoint_Pad_D1.0mm
- removed TP7: CC2, TestPoint:TestPoint_Pad_D1.0mm
- added SW2: Reset, Button_Switch_SMD:SW_SPST_EVQP7A, F.Cu at (161.3, 111.7)
- added TP11: BTN_RESET, TestPoint:TestPoint_Pad_D1.0mm, B.Cu at (158.7, 104.8)
- AE1: footprint TrActor:NFC-Coil -> TrActor:AANI-CH-0029
- AE3: footprint Inductor_SMD:L_1206_3216Metric -> TrActor:ACR0301U
- C41, C42: value 120pF,TBD -> 8pF
- C44, C45: value 47u -> 22u; footprint Capacitor_SMD:CP_Elec_5x5.8 -> Capacitor_SMD:CP_Elec_4x5.4
- J1, TP1, TP10, TP12, TP15, TP16, TP17, TP18, TP19, TP2, TP20, TP21, TP22, TP23, TP24, TP25, TP26, TP27, TP28, TP29, TP3, TP4, TP5, TP8, TP9: moved to B.Cu
- J2: footprint Connector_PinHeader_1.27mm:PinHeader_2x05_P1.27mm_Vertical_SMD -> Connector_PinHeader_1.27mm:PinHeader_2x05_P1.27mm_Vertical
- moved TP10 187.1 mm to (158.7, 102.5), turned to 180 degrees
- moved TP5 174.2 mm to (144.4, 112.3), turned to 180 degrees
- moved TP2 173.5 mm to (155.8, 106.0), turned to 180 degrees
- moved TP3 170.9 mm to (155.8, 108.1), turned to 180 degrees
- moved TP22 170.4 mm to (148.1, 91.8), turned to 180 degrees
- moved TP4 170.3 mm to (155.8, 103.8), turned to 180 degrees
- moved TP9 169.3 mm to (140.9, 95.0), turned to 180 degrees
- moved TP26 169.2 mm to (149.8, 85.7), turned to 180 degrees
- moved TP27 168.9 mm to (152.5, 78.2), turned to 180 degrees
- moved TP18 168.9 mm to (156.9, 99.2), turned to 180 degrees
- moved TP23 168.2 mm to (145.8, 91.8), turned to 180 degrees
- moved TP29 167.6 mm to (151.2, 83.0), turned to 180 degrees
- moved TP19 167.4 mm to (157.7, 96.9), turned to 180 degrees
- moved TP17 167.4 mm to (155.4, 95.8), turned to 180 degrees
- moved TP12 166.3 mm to (140.9, 97.1), turned to 180 degrees
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Connections:
- net /MCU/ANT_BLE renamed /MCU/RF_BLE
- net Net-(AE2-FEED) renamed /MCU/BLE_ANT
- net Net-(AE3-PCB_Trace) renamed /UWB/UWB_ANT
- net Net-(C40-Pad2) renamed /UWB/RF_UWB_AC
- net Net-(J3-D+-PadA6) renamed /USB_D+
- net Net-(J3-D--PadA7) renamed /USB_D-
- net Net-(J4-Pin_1) renamed /BATT_RAW
- net Net-(R11-Pad2) renamed /D+
- net Net-(R12-Pad1) renamed /D-
- AE1 pad 1: Net-(AE1-Pad1) -> /MCU/NFC+
- AE1 pad 2: Net-(AE1-Pad2) -> /MCU/NFC-
- C41 pad 1: Net-(AE1-Pad2) -> /MCU/NFC-
- C42 pad 2: Net-(AE1-Pad1) -> /MCU/NFC+
- U1 pad 31: IMU_INT2 -> IMU_INT1
- U1 pad 32: IMU_INT1 -> IMU_INT2
- U1 pad 34: DW_IRQ -> DW_RST
- U1 pad 35: DW_RST -> DW_WAKEUP
- U1 pad 36: DW_WAKEUP -> DW_IRQ
- U1 pad 4: MOSI -> CS_DW
- U1 pad 6: SCK -> MOSI
- U1 pad 7: CS_DW -> SCK
Routing:
- net VSYS: track 6.09 -> 75.4 mm, vias 1 -> 9
- net VBUS: track 6.08 -> 42.3 mm, vias 1 -> 2
- net GND: track 128.4 -> 162.3 mm, vias 34 -> 68
- net /Power Management/RED: track 1.12 -> 29.5 mm, vias 1 -> 2
- net /MCU/~{RESET}: track 1.21 -> 27.4 mm, vias 0 -> 3
- net /Power Management/YELLOW: track 1.01 -> 25.8 mm, vias 1 -> 2
- net /Power Management/GREEN: track 1.12 -> 22.4 mm, vias 1 -> 2
- net SDA: track 2.89 -> 23.0 mm, vias 0 -> 2
- net SCL: track 2.85 -> 22.7 mm, vias 0 -> 2
- net DW_EXTON: track 2.65 -> 22.0 mm
- net /MCU/SWDIO: track 2.31 -> 21.0 mm, vias 0 -> 1
- net /MCU/SWDCLK: track 2.22 -> 20.3 mm, vias 0 -> 2
- net USB+: track 2.29 -> 19.9 mm
- net USB-: track 1.95 -> 19.4 mm
- net BTN_RESET: track 1.64 -> 18.1 mm, vias 1 -> 2
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- added copper zone on In3.Cu, net +1V8
- added copper zone on In2.Cu, net +2V5
- added copper zone on F.Cu, net GND
- added copper zone on In4.Cu, net GND
Other:
- board size 26 x 60 mm -> 26 x 50 mm
- copper layers 4 -> 6
- board text added: "#are we actually using these lol?"
- board text added: "PLACEHOLDER, THIS THING IS ASS"
- board text added: "TO:DO: - Figure out actually good NFC antenna & place - layout nPM - finalize LED positions - locate test points & tagconnect on back of board - decide on side for programming header (probably front?)"
- board text removed: "TO:DO: - Figure out actually good NFC antenna - increase power trace widths - actual RF trace width calcs - physical layout (buttons, LEDs, etc)"
