File: power.kicad_sch (KiCad schematic)
At the start: 0 parts

Commit message: schematic capture like half done, need to do a lot of the smaller things
Parts:
- added C31, C32: 1u, symbol Device:C_Small
- added C33, C34, C35, C36, C37: 10u, symbol Device:C_Small
- added C38: 0.1u, symbol Device:C_Small
- added C39: 2.2u, symbol Device:C_Small
- added D4: Green, symbol Device:LED_Small
- added D5: Yellow, symbol Device:LED_Small
- added D6: Red, symbol Device:LED_Small
- added L5, L6: 2.2u, symbol Device:L_Small
- added R10: 68k, symbol Device:R_Small_US
- added R7, R8: 10k, symbol Device:R_Small_US
- added R9: 47k, symbol Device:R_Small_US
- added U5: nPM1300, Package_DFN_QFN:QFN-40-1EP_5x5mm_P0.4mm_EP3.6x3.6mm_ThermalVias, symbol TrActor:nPM1300
Connections:
- net +1V8: now also C36.1, C38.1, L5.1, R7.2, R8.2, U5.1 (VOUT1), U5.12 (VDDIO)
- net +2V5: now also C37.1, L6.1, U5.32 (VOUT2)
- new net: R10.1, U5.16 (VSET2)
- new net: R9.1, U5.17 (VSET1)
- new net: D4.1 (K), U5.25 (LED0)
- new net: D5.1 (K), U5.26 (LED1)
- new net: D6.1 (K), U5.27 (LED2)
- new net: L5.2, U5.3 (SW1)
- new net: L6.2, U5.5 (SW2)
- new net +BATT: C39.1, U5.19 (VBAT)
- new net BTN_POWER: U5.15 (SHPHLD)
- new net BTN_RESET: U5.7 (GPIO0)
- new net DW_EXTON: U5.8 (GPIO1)
- new net GND: C31.2, C32.2, C33.2, C34.2, C35.2, C36.2, C37.2, C38.2, C39.2, R10.2, R9.2, U5.2 (PVSS2), U5.28 (VINLDO1), U5.29 (VOUTLDO1), U5.30 (VINLDO2), U5.31 (VOUTLDO2), U5.33 (AVSS)
- new net NTC: U5.18 (NTC)
- new net SCL: R8.1, U5.14 (SCL)
- new net SDA: R7.1, U5.13 (SDA)
- new net USB_CC1: U5.23 (CC1)
- new net USB_CC2: U5.24 (CC2)
- new net VBUS: C32.1, U5.22 (VBUS_OUT)
- new net VSYS: C33.1, C34.1, C35.1, D4.2 (A), D5.2 (A), D6.2 (A), U5.20 (VSYS), U5.4 (PVDD)
- new net VUSB: C31.1, U5.21 (VBUS)
- no-connect marks 0 -> 3
Other:
- note added: "Pg. 50 of DS 47k - 1.8V 68k - 2.5V"
- note added: "TO:DO: - LED Selection - inductor selection - test pads"
- note removed: "TO:DO: - All of it lol"

Commit message: all schematic done but RF
Parts:
- added TP1: VBUS, symbol Connector:TestPoint_Alt
- added TP2: VSYS, symbol Connector:TestPoint_Alt
- added TP3: +1.8V, symbol Connector:TestPoint_Alt
- added TP4: +2.5V, symbol Connector:TestPoint_Alt
- added TP6: CC1, symbol Connector:TestPoint
- added TP7: CC2, symbol Connector:TestPoint
- C31, C32, C38: footprint (none) -> Capacitor_SMD:C_0402_1005Metric
- C33, C34, C35, C36, C37, C39: footprint (none) -> Capacitor_SMD:C_0603_1608Metric
- D4, D5, D6: footprint (none) -> LED_SMD:LED_0603_1608Metric
- L5, L6: footprint (none) -> Inductor_SMD:L_0805_2012Metric
- R10, R7, R8, R9: footprint (none) -> Resistor_SMD:R_0603_1608Metric
Connections:
- net +1V8: now also TP3.1
- net +2V5: now also TP4.1
- net USB_CC1: now also TP6.1
- net USB_CC2: now also TP7.1
- net VBUS: now also TP1.1
- net VSYS: now also TP2.1
Other:
- note added: "TO:DO:"
- note removed: "TO:DO: - LED Selection - inductor selection - test pads"
- moved on the sheet: C39

Commit message: schematic & bom done except for UWB RF
Parts:
- TP1, TP2, TP3, TP4: footprint (none) -> TestPoint:TestPoint_Pad_1.5x1.5mm
- TP6, TP7: footprint (none) -> TestPoint:TestPoint_Pad_D1.5mm
Changed lines of the file:
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@@
 			)
 		)
-		(property "Footprint" ""
+		(property "Footprint" "TestPoint:TestPoint_Pad_1.5x1.5mm"
 			(at 149.86 69.85 0)
 			(hide yes)
@@
 			)
 		)
-		(property "Footprint" ""
+		(property "Footprint" "TestPoint:TestPoint_Pad_1.5x1.5mm"
 			(at 142.24 43.18 0)
 			(hide yes)
@@
 			)
 		)
-		(property "Footprint" ""
+		(property "Footprint" "TestPoint:TestPoint_Pad_D1.5mm"
 			(at 91.44 57.15 0)
 			(hide yes)
@@
 			)
 		)
-		(property "Footprint" ""
+		(property "Footprint" "TestPoint:TestPoint_Pad_1.5x1.5mm"
 			(at 173.99 52.07 0)
 			(hide yes)
@@
 			)
 		)
-		(property "Footprint" ""
+		(property "Footprint" "TestPoint:TestPoint_Pad_1.5x1.5mm"
 			(at 149.86 87.63 0)
 			(hide yes)
@@
 			)
 		)
-		(property "Footprint" ""
+		(property "Footprint" "TestPoint:TestPoint_Pad_D1.5mm"
 			(at 78.74 57.15 0)
 			(hide yes)

Commit message: routing started
Parts:
- added U7: USBLC6-2P6, Package_TO_SOT_SMD:SOT-666, symbol Power_Protection:USBLC6-2P6
- R10, R7, R8, R9: footprint Resistor_SMD:R_0603_1608Metric -> Resistor_SMD:R_0402_1005Metric
- U5: footprint Package_DFN_QFN:QFN-40-1EP_5x5mm_P0.4mm_EP3.6x3.6mm_ThermalVias -> Package_DFN_QFN:QFN-32-1EP_5x5mm_P0.5mm_EP3.45x3.45mm_ThermalVias
Connections:
- net GND: now also U5.6 (PVSS2), U7.2 (GND)
- net USB_CC1: now also U7.1 (I/O1); no longer U5.23 (CC1)
- net USB_CC2: now also U7.3 (I/O2); no longer U5.24 (CC2)
- net GREEN: now reaches D4.1 (K), U5.25 (LED0)
- net YELLOW: now reaches D5.1 (K), U5.26 (LED1)
- net RED: now reaches D6.1 (K), U5.27 (LED2)
- new net: U5.23 (CC1), U7.6 (I/O1)
- new net: U5.24 (CC2), U7.4 (I/O2)
- new net V_PRE: U7.5 (VBUS)
Other:
- moved on the sheet: D4, D5, D6, TP6, TP7

Commit message: routing hell
Parts:
- TP1, TP2, TP3, TP4: footprint TestPoint:TestPoint_Pad_1.5x1.5mm -> TestPoint:TestPoint_Pad_1.0x1.0mm
- TP6, TP7: footprint TestPoint:TestPoint_Pad_D1.5mm -> TestPoint:TestPoint_Pad_D1.0mm
Changed lines of the file:
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@@
 			)
 		)
-		(property "Footprint" "TestPoint:TestPoint_Pad_1.5x1.5mm"
+		(property "Footprint" "TestPoint:TestPoint_Pad_1.0x1.0mm"
 			(at 149.86 69.85 0)
 			(hide yes)
@@
 			)
 		)
-		(property "Footprint" "TestPoint:TestPoint_Pad_1.5x1.5mm"
+		(property "Footprint" "TestPoint:TestPoint_Pad_1.0x1.0mm"
 			(at 142.24 43.18 0)
 			(hide yes)
@@
 			)
 		)
-		(property "Footprint" "TestPoint:TestPoint_Pad_D1.5mm"
+		(property "Footprint" "TestPoint:TestPoint_Pad_D1.0mm"
 			(at 69.85 57.15 0)
 			(hide yes)
@@
 			)
 		)
-		(property "Footprint" "TestPoint:TestPoint_Pad_1.5x1.5mm"
+		(property "Footprint" "TestPoint:TestPoint_Pad_1.0x1.0mm"
 			(at 173.99 52.07 0)
 			(hide yes)
@@
 			)
 		)
-		(property "Footprint" "TestPoint:TestPoint_Pad_1.5x1.5mm"
+		(property "Footprint" "TestPoint:TestPoint_Pad_1.0x1.0mm"
 			(at 149.86 87.63 0)
 			(hide yes)
@@
 			)
 		)
-		(property "Footprint" "TestPoint:TestPoint_Pad_D1.5mm"
+		(property "Footprint" "TestPoint:TestPoint_Pad_D1.0mm"
 			(at 57.15 57.15 0)
 			(hide yes)

Commit message: ready for DR
Parts:
- removed TP6: CC1, TestPoint:TestPoint_Pad_D1.0mm, symbol Connector:TestPoint
- removed TP7: CC2, TestPoint:TestPoint_Pad_D1.0mm, symbol Connector:TestPoint
Other:
- moved on the sheet: U7
Changed lines of the file:
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@@
 	)
 	(junction
-		(at 64.77 60.96)
-		(diameter 0)
-		(color 0 0 0 0)
-	)
-	(junction
 		(at 147.32 87.63)
 		(diameter 0)
@@
 	)
 	(junction
-		(at 62.23 58.42)
-		(diameter 0)
-		(color 0 0 0 0)
-	)
-	(junction
 		(at 146.05 121.92)
 		(diameter 0)
@@
 	(wire
 		(pts
-			(xy 54.61 60.96) (xy 64.77 60.96)
-		)
-		(stroke
-			(width 0)
-			(type default)
-		)
-	)
-	(wire
-		(pts
 			(xy 88.9 128.27) (xy 88.9 129.54)
 		)
@@
 	(wire
 		(pts
-			(xy 82.55 66.04) (xy 82.55 67.31)
+			(xy 74.93 66.04) (xy 74.93 67.31)
 		)
 		(stroke
@@
 	(wire
 		(pts
-			(xy 62.23 58.42) (xy 77.47 58.42)
+			(xy 54.61 58.42) (xy 69.85 58.42)
 		)
 		(stroke
@@
 	(wire
 		(pts
-			(xy 87.63 58.42) (xy 110.49 58.42)
-		)
-		(stroke
-			(width 0)
-			(type default)
-		)
-	)
-	(wire
-		(pts
 			(xy 146.05 105.41) (xy 146.05 107.95)
 		)
@@
 	(wire
 		(pts
-			(xy 82.55 44.45) (xy 82.55 53.34)
+			(xy 74.93 44.45) (xy 74.93 53.34)
 		)
 		(stroke
@@
 	(wire
 		(pts
-			(xy 54.61 58.42) (xy 62.23 58.42)
-		)
-		(stroke
-			(width 0)
-			(type default)
-		)
-	)
-	(wire
-		(pts
 			(xy 157.48 52.07) (xy 162.56 52.07)
 		)
@@
 	(wire
 		(pts
-			(xy 64.77 60.96) (xy 77.47 60.96)
+			(xy 54.61 60.96) (xy 69.85 60.96)
 		)
 		(stroke
@@
 	(wire
 		(pts
-			(xy 62.23 57.15) (xy 62.23 58.42)
+			(xy 104.14 55.88) (xy 110.49 55.88)
 		)
 		(stroke
@@
 	(wire
 		(pts
-			(xy 104.14 55.88) (xy 110.49 55.88)
+			(xy 100.33 52.07) (xy 100.33 50.8)
 		)
 		(stroke
@@
 	(wire
 		(pts
-			(xy 100.33 52.07) (xy 100.33 50.8)
+			(xy 88.9 129.54) (xy 88.9 130.81)
 		)
 		(stroke
@@
 	(wire
 		(pts
-			(xy 88.9 129.54) (xy 88.9 130.81)
+			(xy 80.01 58.42) (xy 110.49 58.42)
 		)
 		(stroke
@@
 	(wire
 		(pts
-			(xy 64.77 57.15) (xy 64.77 60.96)
-		)
-		(stroke
-			(width 0)
-			(type default)
-		)
-	)
-	(wire
-		(pts
 			(xy 97.79 68.58) (xy 110.49 68.58)
 		)
@@
 	(wire
 		(pts
-			(xy 88.9 93.98) (xy 110.49 93.98)
+			(xy 80.01 60.96) (xy 110.49 60.96)
 		)
 		(stroke
@@
 	(wire
 		(pts
-			(xy 147.32 92.71) (xy 147.32 93.98)
+			(xy 88.9 93.98) (xy 110.49 93.98)
 		)
 		(stroke
@@
 	(wire
 		(pts
-			(xy 87.63 60.96) (xy 110.49 60.96)
+			(xy 147.32 92.71) (xy 147.32 93.98)
 		)
 		(stroke
@@
 	(global_label "V_PRE"
 		(shape input)
-		(at 82.55 44.45 90)
+		(at 74.93 44.45 90)
 		(fields_autoplaced yes)
 		(effects
@@
 		)
 		(property "Intersheetrefs" "${INTERSHEET_REFS}"
-			(at 82.55 36.3738 90)
+			(at 74.93 36.3738 90)
 			(hide yes)
 			(show_name no)
@@
 	(symbol
 		(lib_id "Power_Protection:USBLC6-2P6")
-		(at 82.55 58.42 0)
+		(at 74.93 58.42 0)
 		(unit 1)
 		(body_style 1)
@@
 		(dnp no)
 		(property "Reference" "U7"
-			(at 83.058 54.356 0)
+			(at 75.438 54.356 0)
 			(show_name no)
 			(do_not_autoplace no)
@@
 		)
 		(property "Value" "USBLC6-2P6"
-			(at 85.598 63.754 90)
+			(at 77.978 63.754 90)
 			(show_name no)
 			(do_not_autoplace no)
@@
 		)
 		(property "Footprint" "Package_TO_SOT_SMD:SOT-666"
-			(at 83.566 65.151 0)
+			(at 75.946 65.151 0)
 			(hide yes)
 			(show_name no)
@@
 		)
 		(property "Datasheet" "https://www.st.com/resource/en/datasheet/usblc6-2.pdf"
-			(at 83.566 67.056 0)
+			(at 75.946 67.056 0)
 			(hide yes)
 			(show_name no)
@@
 		)
 		(property "Description" "Very low capacitance ESD protection diode, 2 data-line, SOT-666"
-			(at 82.55 58.42 0)
+			(at 74.93 58.42 0)
 			(hide yes)
 			(show_name no)
@@
 	)
 	(symbol
-		(lib_id "Connector:TestPoint")
-		(at 64.77 57.15 0)
-		(unit 1)
-		(body_style 1)
-		(exclude_from_sim no)
-		(in_bom yes)
-		(on_board yes)
-		(in_pos_files yes)
-		(dnp no)
-		(fields_autoplaced yes)
-		(property "Reference" "TP7"
-			(at 67.31 52.5779 0)
-			(show_name no)
-			(do_not_autoplace no)
-			(effects
-				(font
-					(size 1.27 1.27)
-				)
-				(justify left)
-			)
-		)
-		(property "Value" "CC2"
-			(at 67.31 55.1179 0)
-			(show_name no)
-			(do_not_autoplace no)
-			(effects
-				(font
-					(size 1.27 1.27)
-				)
-				(justify left)
-			)
-		)
-		(property "Footprint" "TestPoint:TestPoint_Pad_D1.0mm"
-			(at 69.85 57.15 0)
-			(hide yes)
-			(show_name no)
-			(do_not_autoplace no)
-			(effects
-				(font
-					(size 1.27 1.27)
-				)
-			)
-		)
-		(property "Datasheet" ""
-			(at 69.85 57.15 0)
-			(hide yes)
-			(show_name no)
-			(do_not_autoplace no)
-			(effects
-				(font
-					(size 1.27 1.27)
-				)
-			)
-		)
-		(property "Description" "test point"
-			(at 64.77 57.15 0)
-			(hide yes)
-			(show_name no)
-			(do_not_autoplace no)
-			(effects
-				(font
-					(size 1.27 1.27)
-				)
-			)
-		)
-		(pin "1"
-		)
-		(instances
-			(project "TrActor-Board"
-				(path "/e63e39d7-6ac0-4ffd-8aa3-1841a4541b55/e82fad38-4c10-4679-a703-07ea413d1661"
-					(reference "TP7")
-					(unit 1)
-				)
-			)
-		)
-	)
-	(symbol
 		(lib_id "power:GND")
 		(at 146.05 109.22 0)
@@
 	(symbol
 		(lib_id "power:GND")
-		(at 82.55 67.31 0)
+		(at 74.93 67.31 0)
 		(unit 1)
 		(body_style 1)
@@
 		(dnp no)
 		(property "Reference" "#PWR072"
-			(at 82.55 73.66 0)
+			(at 74.93 73.66 0)
 			(hide yes)
 			(show_name no)
@@
 		)
 		(property "Value" "GND"
-			(at 82.55 71.12 0)
+			(at 74.93 71.12 0)
 			(show_name no)
 			(do_not_autoplace no)
@@
 		)
 		(property "Footprint" ""
-			(at 82.55 67.31 0)
+			(at 74.93 67.31 0)
 			(hide yes)
 			(show_name no)
@@
 		)
 		(property "Datasheet" ""
-			(at 82.55 67.31 0)
+			(at 74.93 67.31 0)
 			(hide yes)
 			(show_name no)
@@
 		)
 		(property "Description" "Power symbol creates a global label with name \"GND\" , ground"
-			(at 82.55 67.31 0)
+			(at 74.93 67.31 0)
 			(hide yes)
 			(show_name no)
@@
 					(unit 1)
 				)
-			)
-		)
-	)
-	(symbol
-		(lib_id "Connector:TestPoint")
-		(at 62.23 57.15 0)
-		(mirror y)
-		(unit 1)
-		(body_style 1)
-		(exclude_from_sim no)
-		(in_bom yes)
-		(on_board yes)
-		(in_pos_files yes)
-		(dnp no)
-		(property "Reference" "TP6"
-			(at 59.69 52.5779 0)
-			(show_name no)
-			(do_not_autoplace no)
-			(effects
-				(font
-					(size 1.27 1.27)
-				)
-				(justify left)
-			)
-		)
-		(property "Value" "CC1"
-			(at 59.69 55.1179 0)
-			(show_name no)
-			(do_not_autoplace no)
-			(effects
-				(font
-					(size 1.27 1.27)
-				)
-				(justify left)
-			)
-		)
-		(property "Footprint" "TestPoint:TestPoint_Pad_D1.0mm"
-			(at 57.15 57.15 0)
-			(hide yes)
-			(show_name no)
-			(do_not_autoplace no)
-			(effects
-				(font
-					(size 1.27 1.27)
-				)
-			)
-		)
-		(property "Datasheet" ""
-			(at 57.15 57.15 0)
-			(hide yes)
-			(show_name no)
-			(do_not_autoplace no)
-			(effects
-				(font
-					(size 1.27 1.27)
-				)
-			)
-		)
-		(property "Description" "test point"
-			(at 62.23 57.15 0)
-			(hide yes)
-			(show_name no)
-			(do_not_autoplace no)
-			(effects
-				(font
-					(size 1.27 1.27)
-				)
-			)
-		)
-		(pin "1"
-		)
-		(instances
-			(project "TrActor-Board"
-				(path "/e63e39d7-6ac0-4ffd-8aa3-1841a4541b55/e82fad38-4c10-4679-a703-07ea413d1661"
-					(reference "TP6")
-					(unit 1)
-				)

Commit message: mag added. ready for order?
Parts:
- R7, R8: value 10k -> 2.7k
Changed lines of the file:
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@@
 			)
 		)
-		(property "Value" "10k"
+		(property "Value" "2.7k"
 			(at 97.79 120.6499 0)
 			(show_name no)
@@
 			)
 		)
-		(property "Value" "10k"
+		(property "Value" "2.7k"
 			(at 106.68 123.1899 0)
 			(show_name no)

Commit message: ordering commit fr
Parts:
- TP1, TP2, TP3, TP4: now left out of the parts list
Changed lines of the file:
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@@
 		(body_style 1)
 		(exclude_from_sim no)
-		(in_bom yes)
+		(in_bom no)
 		(on_board yes)
 		(in_pos_files yes)
@@
 		(body_style 1)
 		(exclude_from_sim no)
-		(in_bom yes)
+		(in_bom no)
 		(on_board yes)
 		(in_pos_files yes)
@@
 		(body_style 1)
 		(exclude_from_sim no)
-		(in_bom yes)
+		(in_bom no)
 		(on_board yes)
 		(in_pos_files yes)
@@
 		(body_style 1)
 		(exclude_from_sim no)
-		(in_bom yes)
-		(on_board yes)
-		(in_pos_files yes)
+		(in_bom no)
+		(on_board yes)
+		(in_pos_files yes)
